Commit message: Revised/working plotting scripts and such

File: robots/spot/spot.urdf (robot description, URDF)
Before this commit: robot spot, 17 links, 16 joints
Links:
- link fl.foot: mass None -> 0.200
- link fr.foot: mass None -> 0.200
- link hl.foot: mass None -> 0.200
- link hr.foot: mass None -> 0.200
